File: hardware/kicad/Orpheus.kicad_sch (KiCad schematic)
At the start: 0 parts

Commit message: Added Symbols & Footprints of SD Module, ESP32 & Screw Terminal Block
Parts:
- added J1: Screw Terminal Block 1x2, Orpheus:ScrewTerminal_1x2, symbol Orpheus:ScrewTerminal_1x2
- added J2: MicroSD Card, Orpheus:MicroSD_Card, symbol Orpheus:MicroSD_Card
- added U1: ESP32-S3 DevBoard, Orpheus:ESP32-S3 DevBoard, symbol Orpheus:ESP32_S3_DevBoard
Connections:
- new net 3V3: J2.4 (VDD), U1.1 (3V3), U1.2 (3V3)
- new net 8V4: J1.1
- new net COVER_GND: J1.2, J2.6 (VSS), J2.G1 (COVER_GND), J2.G2 (COVER_GND), J2.G3 (COVER_GND), J2.G4 (COVER_GND), U1.22 (GND), U1.43 (GND), U1.44 (GND)
- new net SD_CS: J2.2 (CD/DAT3), U1.32 (38)
- new net SD_MISO: J2.7 (DAT0), U1.33 (37)
- new net SD_MOSI: J2.3 (CMD), U1.35
- new net SD_SCLK: J2.5 (CLK), U1.34 (36)
- no-connect marks 0 -> 3
Other:
- note added: "ESP32-S3 DEVELOPMENT BOARD"
- note added: "INPUT CONNECTORS"
